Commit message: Add runnable RDSim runtime files

File: rdsim_description/urdf/rdsim.gazebo.xacro (robot description, xacro)
@@ -7,5 +7,4 @@
     <material>Gazebo/Grey</material>
   </gazebo>
-<!-- wheel -->
   <gazebo reference="wheel_left_link">
     <mu1>10000000</mu1>
@@ -28,5 +27,4 @@
     <material>Gazebo/FlatBlack</material>
   </gazebo>
-<!-- caster -->
   <gazebo reference="caster_link">
     <mu1>0.1</mu1>
@@ -38,5 +36,4 @@
     <material>Gazebo/FlatBlack</material>
   </gazebo>
-<!-- imu -->
   <gazebo reference="imu_link">
     <material>Gazebo/Yellow</material>
@@ -44,5 +41,4 @@
       <plugin filename="libgazebo_ros_imu_sensor.so" name="imu_plugin">
         <ros>
-          <!-- <namespace>/demo</namespace> -->
           <remapping>~/out:=imu</remapping>
         </ros>
@@ -108,5 +104,4 @@
     </sensor>
   </gazebo>
-<!-- differential type config -->
   <gazebo>
     <plugin name='diff_drive' filename='libgazebo_ros_diff_drive.so'>
@@ -203,10 +198,10 @@
       <pose>0 0 0 0 0 0</pose>
       <always_on>false</always_on>
-      <update_rate>10.0</update_rate> <!-- 업데이트 속도 줄임 -->
-      <visualize>false</visualize> <!-- 비주얼라이제이션 비활성화 -->
+      <update_rate>10.0</update_rate>
+      <visualize>false</visualize>
       <ray>
         <scan>
           <horizontal>
-            <samples>360</samples> <!-- 가로 샘플 수 줄임 -->
+            <samples>360</samples>
             <resolution>1</resolution>
             <min_angle>-3.14159</min_angle>
@@ -214,5 +209,5 @@
           </horizontal>
           <vertical>
-            <samples>32</samples> <!-- 수직 샘플 수 줄임 -->
+            <samples>32</samples>
             <resolution>1</resolution>
             <min_angle>-0.561799</min_angle>
@@ -222,8 +217,7 @@
         <range>
           <min>0.30</min>
-          <max>50.0</max> <!-- 범위 줄임 -->
+          <max>50.0</max>
           <resolution>0.01</resolution>
         </range>
-        <!-- 소음 설정 제거 -->
       </ray>
       <plugin name="gazebo_ros_ray_sensor" filename="libgazebo_ros_ray_sensor.so">
@@ -237,5 +231,4 @@
     </sensor>
   </gazebo>
-  <!-- GPS -->
   <gazebo reference="gps_link">
     <sensor name="gps_sensor" type="gps">
@@ -247,5 +240,4 @@
         <output_type>sensor_msgs/NavSatFix</output_type>
         <frame_name>gps_link</frame_name>
-        <!-- 임의의 위도, 경도 값 설정 -->
         <latitude_deg>37.466</latitude_deg>
         <longitude_deg>126.932</longitude_deg>
@@ -257,6 +249,6 @@
         <position_sensing>
           <noise type="gaussian">
-            <mean>0.0</mean> <!-- 기본적으로 노이즈가 없는 설정 -->
-            <stddev>0.0</stddev> <!-- 노이즈 표준편차 설정 -->
+            <mean>0.0</mean>
+            <stddev>0.0</stddev>
           </noise>
         </position_sensing>
@@ -264,6 +256,4 @@
     </sensor>
   </gazebo>
-<!-- 카메라 플러그인 추가 -->
-<!-- Front-right camera -->
 <gazebo reference="camera_front_right_link">
   <sensor type="camera" name="camera_front_right_sensor">
@@ -292,5 +282,4 @@
   </sensor>
 </gazebo>
-<!-- Front-left camera -->
 <gazebo reference="camera_front_left_link">
   <sensor type="camera" name="camera_front_left_sensor">
@@ -319,5 +308,4 @@
   </sensor>
 </gazebo>
-<!-- Back-right camera -->
 <gazebo reference="camera_back_right_link">
   <sensor type="camera" name="camera_back_right_sensor">
@@ -346,5 +334,4 @@
   </sensor>
 </gazebo>
-<!-- Back-left camera -->
 <gazebo reference="camera_back_left_link">
   <sensor type="camera" name="camera_back_left_sensor">
@@ -373,5 +360,4 @@
   </sensor>
 </gazebo>
-<!-- camera_top_link -->
 <gazebo reference="camera_top_link">
   <sensor type="camera" name="camera_top_sensor">

File: rdsim_description/urdf/rdsim.urdf.xacro (robot description, xacro)
@@ -1,6 +1,4 @@
 <?xml version="1.0"?>
 <robot name="rdsim" xmlns:xacro="http://ros.org/wiki/xacro">
-  <!-- <xacro:arg name="prefix" default="" /> -->
-  <!-- Define robot constants -->
   <xacro:property name="base_width" value="0.62"/>
   <xacro:property name="base_length" value="0.82"/>
@@ -12,5 +10,4 @@
   <xacro:property name="wheel_xoff" value="0.24"/>
   <xacro:property name="caster_xoff" value="0.28"/>
-  <!-- Define some commonly used intertial properties  -->
   <xacro:macro name="box_inertia" params="m w h d">
     <inertial>
@@ -33,5 +30,4 @@
     </inertial>
   </xacro:macro>
-   <!-- Robot Footprint -->
   <link name="base_footprint">
   	<xacro:box_inertia m="0" w="0" d="0" h="0"/>
@@ -42,5 +38,4 @@
     <origin xyz="${-1 * wheel_xoff} 0.0 ${(wheel_radius+wheel_zoff)}" rpy="0 0 0"/>
   </joint>
-  <!-- Robot Base -->
   <link name="base_link">
     <visual>
@@ -59,5 +54,4 @@
     <xacro:box_inertia m="15" w="${base_width}" d="${base_length}" h="${base_height}"/>
   </link>
-<!-- gps link -->
   <link name="gps_link">
     <visual>
@@ -67,5 +61,4 @@
     </visual>
   </link>
-  <!-- gps joint -->
   <joint name="gps_joint" type="fixed">
     <parent link="base_footprint"/>
@@ -233,5 +226,4 @@
     <origin xyz="0.215 0 0.05" rpy="0 0 0"/>
   </joint>
-  <!-- Add four cameras positioned diagonally at 45-degree angles -->
   <xacro:macro name="add_camera" params="name x y z roll pitch yaw">
     <link name="${name}_link">
@@ -242,15 +234,4 @@
         </geometry>
       </visual>
-      <!-- <collision>
-        <origin xyz="0 0 0" rpy="0 0 0"/>
-        <geometry>
-          <box size="0.015 0.130 0.022"/>
-        </geometry>
-      </collision> -->
-      <!-- <inertial>
-        <origin xyz="0 0 0" rpy="0 0 0"/>
-        <mass value="0.035"/>
-        <inertia ixx="0.001" ixy="0" ixz="0" iyy="0.001" iyz="0" izz="0.001"/>
-      </inertial> -->
     </link>
     <joint name="${name}_joint" type="fixed">
@@ -260,11 +241,4 @@
     </joint>
   </xacro:macro>
-  <!-- Adding four cameras in diagonal directions -->
-  <!--xacro:add_camera name="camera_front_right" x="0.25" y="0.25" z="0.25" roll="0" pitch="0" yaw="${pi/4}"/>
-  <xacro:add_camera name="camera_front_left" x="0.25" y="-0.25" z="0.25" roll="0" pitch="0" yaw="${-pi/4}"/>
-  <xacro:add_camera name="camera_back_right" x="-0.25" y="0.25" z="0.25" roll="0" pitch="0" yaw="${3*pi/4}"/>
-  <xacro:add_camera name="camera_back_left" x="-0.25" y="-0.25" z="0.25" roll="0" pitch="0" yaw="${-3*pi/4}"/>
-  <xacro:add_camera name="camera_top" x="0" y="0" z="5.25" roll="0" pitch="${pi/2}" yaw="0"/-->
-  <!-- Include gazebo macro -->
   <xacro:include filename="$(find rdsim_description)/urdf/rdsim.gazebo.xacro" />
 </robot>
